File: X15-Conversion.sch (EAGLE design)
At the start: 22 parts, among them U2 LINEAR,AZ1117CR-3.3TRG1DIODES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

Commit message: Second commit to board review
Parts:
- added D1: Yellow, SparkFun-LED:LED-YELLOW0603
- added D3: BLUE, SparkFun-LED:LED-BLUE0603
- added D5: RED, SparkFun-LED:LED-RED0603
- added R4: 20, SparkFun-Resistors:20OHM-0603-1/10W-1%
- added R5, R6: 100, SparkFun-Resistors:20OHM-0603-1/10W-1%
Connections:
- new net N$2: D1.A, R4.1
- new net N$5: D5.A, R5.1
- new net N$6: D3.A, R6.1
- net 12V: now also R4.2
- net 3.3V: now also R6.2
- net 5.2V: now also R5.2
- net GND: now also D1.C, D3.C, D5.C
Other:
- moved on the sheet: C1, C10, C11, C2, C4, C7, C8, C9, CONN, D2, L2, R1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

Commit message: added some cool files
Parts:
- removed CONN: CONVERSION-DISTRIBUTION, CONN, Distribution-Conversion (3):CONVERSION-DISTRIBUTION
- removed D1: Yellow, SparkFun-LED:LED-YELLOW0603
- removed D3: BLUE, SparkFun-LED:LED-BLUE0603
- removed D5: RED, SparkFun-LED:LED-RED0603
- removed R4: 20, SparkFun-Resistors:20OHM-0603-1/10W-1%
- removed R5, R6: 100, SparkFun-Resistors:20OHM-0603-1/10W-1%
- removed U$2: 3.3V_TESTPOINT, testpoints:3.3V_TESTPOINT
- removed U$3: 5.2V_TESTPOINT, testpoints:5.2V_TESTPOINT
- removed U$4: 12V_TESTPOINT, testpoints:12V_TESTPOINT
- removed U$5, U$6, U$7: GND_TESTPOINT, testpoints:GND_TESTPOINT
- added CONN1: CONVERSION-DISTRIBUTION, CONN, Distribution-Conversion (3):CONVERSION-DISTRIBUTION
- added D4: Yellow, SparkFun-LED:LED-YELLOW0603
- added D6: RED, SparkFun-LED:LED-RED0603
- added D7: BLUE, SparkFun-LED:LED-BLUE0603
- added R7, R8, R9: 150, SparkFun-Resistors:20OHM-0603-1/10W-1%
- added U$10: 12V_TESTPOINT, testpoints:12V_TESTPOINT
- added U$11, U$12, U$13: GND_TESTPOINT, testpoints:GND_TESTPOINT
- added U$8: 3.3V_TESTPOINT, testpoints:3.3V_TESTPOINT
- added U$9: 5.2V_TESTPOINT, testpoints:5.2V_TESTPOINT
Connections:
- removed net N$2: D1.A, R4.1
- removed net N$5: D5.A, R5.1
- removed net N$6: D3.A, R6.1
- new net N$10: D7.A, R9.1
- new net N$8: D4.A, R7.1
- new net N$9: D6.A, R8.1
- net 12V: now also CONN1.VIN+, R7.2, U$10.12V; no longer CONN.VIN+, R4.2, U$4.12V
- net 3.3V: now also CONN1.VOUT+_3, R9.2, U$8.3.3V; no longer CONN.VOUT+_3, R6.2, U$2.3.3V
- net 5.2V: now also CONN1.VOUT+_5, R8.2, U$9.5.2V; no longer CONN.VOUT+_5, R5.2, U$3.5.2V
- net GND: now also CONN1.VIN-, CONN1.VOUT-, D4.C, D6.C, D7.C, U$11.GND, U$12.GND, U$13.GND; no longer CONN.VIN-, CONN.VOUT-, D1.C, D3.C, D5.C, U$5.GND, U$6.GND, U$7.GND
Other:
- note added: "Test Voltage LEDs"
