File: X15-Conversion.sch (EAGLE design)
At the start: 31 parts, among them U1 LINEAR,AZ1117CR-3.3TRG1DIODES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

Commit message: Changed the fonts
Parts:
- removed U$13: GND_TESTPOINT, X15-Conversion-Parts-Library:GND_TESTPOINT
- renumbered J1 to GND
Connections:
- net GND: no longer U$13.GND
Changed lines of the file:
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@@
 <part name="U$11" library="X15-Conversion-Parts-Library" deviceset="GND_TESTPOINT" device=""/>
 <part name="U$12" library="X15-Conversion-Parts-Library" deviceset="GND_TESTPOINT" device=""/>
-<part name="U$13" library="X15-Conversion-Parts-Library" deviceset="GND_TESTPOINT" device=""/>
 <part name="CONN1" library="X15-Conversion-Parts-Library" deviceset="CONVERSION-DISTRIBUTION" device=""/>
 <part name="D4" library="SparkFun-LED" library_urn="urn:adsk.eagle:library:529" deviceset="LED-YELLOW" device="0603" package3d_urn="urn:adsk.eagle:package:39354/1" value="Yellow"/>
@@
 <part name="COUT3" library="X15-Conversion-Parts-Library" deviceset="C-TANTALUM(10UF_150UF)" device="" package3d_urn="urn:adsk.eagle:package:25131320/3" value="150uF"/>
 <part name="L1" library="X15-Conversion-Parts-Library" deviceset="HCMA1305" device="" package3d_urn="urn:adsk.eagle:package:24201702/2" value="15uH"/>
-<part name="J1" library="SparkFun-Connectors" library_urn="urn:adsk.eagle:library:513" deviceset="CONN_02" device="" package3d_urn="urn:adsk.eagle:package:38039/1"/>
+<part name="GND" library="SparkFun-Connectors" library_urn="urn:adsk.eagle:library:513" deviceset="CONN_02" device="" package3d_urn="urn:adsk.eagle:package:38039/1"/>
 <part name="J2" library="SparkFun-Connectors" library_urn="urn:adsk.eagle:library:513" deviceset="CONN_02" device="" package3d_urn="urn:adsk.eagle:package:38039/1"/>
 <part name="J3" library="SparkFun-Connectors" library_urn="urn:adsk.eagle:library:513" deviceset="CONN_02" device="" package3d_urn="urn:adsk.eagle:package:38039/1"/>
@@
 <instance part="U$11" gate="G$1" x="-81.28" y="-38.1" smashed="yes"/>
 <instance part="U$12" gate="G$1" x="-81.28" y="-48.26" smashed="yes"/>
-<instance part="U$13" gate="G$1" x="-81.28" y="-58.42" smashed="yes"/>
 <instance part="CONN1" gate="G$1" x="58.42" y="-17.78" smashed="yes">
 <attribute name="NAME" x="50.8" y="-10.16" size="1.778" layer="95"/>
@@
 <attribute name="VALUE" x="-53.848" y="40.005" size="1.778" layer="96" font="vector" rot="R180" align="top-left"/>
 </instance>
-<instance part="J1" gate="G$1" x="68.58" y="71.12" smashed="yes">
+<instance part="GND" gate="G$1" x="68.58" y="71.12" smashed="yes">
 <attribute name="VALUE" x="66.04" y="66.294" size="1.778" layer="96" font="vector"/>
 <attribute name="NAME" x="66.04" y="76.708" size="1.778" layer="95" font="vector"/>
@@
 </segment>
 <segment>
-<pinref part="U$13" gate="G$1" pin="GND"/>
-<wire x1="-76.2" y1="-58.42" x2="-66.04" y2="-58.42" width="0.1524" layer="91"/>
-<label x="-66.04" y="-58.42" size="1.778" layer="95" xref="yes"/>
-</segment>
-<segment>
 <pinref part="CONN1" gate="G$1" pin="VIN-"/>
 <wire x1="45.72" y1="-17.78" x2="35.56" y2="-17.78" width="0.1524" layer="91"/>
@@
 </segment>
 <segment>
-<pinref part="J1" gate="G$1" pin="2"/>
+<pinref part="GND" gate="G$1" pin="2"/>
 <wire x1="76.2" y1="73.66" x2="88.9" y2="73.66" width="0.1524" layer="91"/>
 <label x="86.36" y="73.66" size="1.778" layer="95" align="bottom-right"/>
 </segment>
 <segment>
-<pinref part="J1" gate="G$1" pin="1"/>
+<pinref part="GND" gate="G$1" pin="1"/>
 <wire x1="76.2" y1="71.12" x2="88.9" y2="71.12" width="0.1524" layer="91"/>
 <label x="86.36" y="71.12" size="1.778" layer="95" align="bottom-right"/>

Commit message: Added labels to the lights
Parts:
- renumbered D4 to 12V, D6 to 5.2V, D7 to 3.3V
Changed lines of the file:
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@@
 <part name="U$12" library="X15-Conversion-Parts-Library" deviceset="GND_TESTPOINT" device=""/>
 <part name="CONN1" library="X15-Conversion-Parts-Library" deviceset="CONVERSION-DISTRIBUTION" device=""/>
-<part name="D4" library="SparkFun-LED" library_urn="urn:adsk.eagle:library:529" deviceset="LED-YELLOW" device="0603" package3d_urn="urn:adsk.eagle:package:39354/1" value="Yellow"/>
+<part name="12V" library="SparkFun-LED" library_urn="urn:adsk.eagle:library:529" deviceset="LED-YELLOW" device="0603" package3d_urn="urn:adsk.eagle:package:39354/1" value="Yellow"/>
 <part name="R7" library="SparkFun-Resistors" library_urn="urn:adsk.eagle:library:532" deviceset="20OHM" device="-0603-1/10W-1%" package3d_urn="urn:adsk.eagle:package:39650/1" value="600"/>
 <part name="R8" library="SparkFun-Resistors" library_urn="urn:adsk.eagle:library:532" deviceset="20OHM" device="-0603-1/10W-1%" package3d_urn="urn:adsk.eagle:package:39650/1" value="300"/>
 <part name="R9" library="SparkFun-Resistors" library_urn="urn:adsk.eagle:library:532" deviceset="20OHM" device="-0603-1/10W-1%" package3d_urn="urn:adsk.eagle:package:39650/1" value="200"/>
 <part name="FRAME3" library="frames" library_urn="urn:adsk.eagle:library:229" deviceset="A4L-LOC" device="" value="2"/>
-<part name="D6" library="SparkFun-LED" library_urn="urn:adsk.eagle:library:529" deviceset="LED-RED" device="0603" package3d_urn="urn:adsk.eagle:package:39354/1" value="RED"/>
-<part name="D7" library="SparkFun-LED" library_urn="urn:adsk.eagle:library:529" deviceset="LED-BLUE" device="0603" package3d_urn="urn:adsk.eagle:package:39354/1" value="BLUE"/>
+<part name="5.2V" library="SparkFun-LED" library_urn="urn:adsk.eagle:library:529" deviceset="LED-RED" device="0603" package3d_urn="urn:adsk.eagle:package:39354/1" value="RED"/>
+<part name="3.3V" library="SparkFun-LED" library_urn="urn:adsk.eagle:library:529" deviceset="LED-BLUE" device="0603" package3d_urn="urn:adsk.eagle:package:39354/1" value="BLUE"/>
 <part name="CIN1" library="X15-Conversion-Parts-Library" deviceset="EEEFKE181XSP" device="" value="180uF"/>
 <part name="U1" library="X15-Conversion-Parts-Library" deviceset="LINEAR,AZ1117CR-3.3TRG1" device="DIODES_AZ1117CH-3.3TRG1_0_0"/>
@@
 <attribute name="NAME" x="50.8" y="-10.16" size="1.778" layer="95"/>
 </instance>
-<instance part="D4" gate="G$1" x="-58.42" y="63.5" smashed="yes" rot="R90">
+<instance part="12V" gate="G$1" x="-58.42" y="63.5" smashed="yes" rot="R90">
 <attribute name="NAME" x="-53.848" y="60.071" size="1.778" layer="95" font="vector" rot="R180"/>
 <attribute name="VALUE" x="-53.848" y="65.405" size="1.778" layer="96" font="vector" rot="R180" align="top-left"/>
@@
 <attribute name="SHEET" x="116.205" y="-78.74" size="2.54" layer="94"/>
 </instance>
-<instance part="D6" gate="G$1" x="-58.42" y="50.8" smashed="yes" rot="R90">
+<instance part="5.2V" gate="G$1" x="-58.42" y="50.8" smashed="yes" rot="R90">
 <attribute name="NAME" x="-53.848" y="47.371" size="1.778" layer="95" font="vector" rot="R180"/>
 <attribute name="VALUE" x="-53.848" y="52.705" size="1.778" layer="96" font="vector" rot="R180" align="top-left"/>
 </instance>
-<instance part="D7" gate="G$1" x="-58.42" y="38.1" smashed="yes" rot="R90">
+<instance part="3.3V" gate="G$1" x="-58.42" y="38.1" smashed="yes" rot="R90">
 <attribute name="NAME" x="-53.848" y="34.671" size="1.778" layer="95" font="vector" rot="R180"/>
 <attribute name="VALUE" x="-53.848" y="40.005" size="1.778" layer="96" font="vector" rot="R180" align="top-left"/>
@@
 </segment>
 <segment>
-<pinref part="D4" gate="G$1" pin="C"/>
+<pinref part="12V" gate="G$1" pin="C"/>
 <wire x1="-53.34" y1="63.5" x2="-43.18" y2="63.5" width="0.1524" layer="91"/>
 <label x="-43.18" y="63.5" size="1.778" layer="95" xref="yes"/>
@@
 <wire x1="-53.34" y1="50.8" x2="-43.18" y2="50.8" width="0.1524" layer="91"/>
 <label x="-43.18" y="50.8" size="1.778" layer="95" xref="yes"/>
-<pinref part="D6" gate="G$1" pin="C"/>
+<pinref part="5.2V" gate="G$1" pin="C"/>
 </segment>
 <segment>
 <wire x1="-53.34" y1="38.1" x2="-43.18" y2="38.1" width="0.1524" layer="91"/>
 <label x="-43.18" y="38.1" size="1.778" layer="95" xref="yes"/>
-<pinref part="D7" gate="G$1" pin="C"/>
+<pinref part="3.3V" gate="G$1" pin="C"/>
 </segment>
 <segment>
@@
 <net name="N$8" class="0">
 <segment>
-<pinref part="D4" gate="G$1" pin="A"/>
+<pinref part="12V" gate="G$1" pin="A"/>
 <pinref part="R7" gate="G$1" pin="1"/>
 </segment>
@@
 <segment>
 <pinref part="R8" gate="G$1" pin="1"/>
-<pinref part="D6" gate="G$1" pin="A"/>
+<pinref part="5.2V" gate="G$1" pin="A"/>
 </segment>
 </net>
@@
 <segment>
 <pinref part="R9" gate="G$1" pin="1"/>
-<pinref part="D7" gate="G$1" pin="A"/>
-</segment>
-</net>
+<pinref part="3.3V" gate="G$1" pin="A"/>
+</segment>
+</net>
