File: X15-Conversion.brd (EAGLE design)
At the start: 50.8 x 62.9 mm, 28 parts, among them U1 LINEAR,AZ1117CR-3.3TRG1DIODES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

Commit message: Finalized Board for Review
Parts:
- moved D7 4.02 mm to (11.4, 10.2)
- moved C10 1.27 mm to (3.17, 24.1)
Routing:
- net 5.2V: track 97.2 -> 93.3 mm
- net N$10: track 6.69 -> 9.46 mm
- net 3.3V: track 73.2 -> 73.9 mm

Commit message: Edited suggestions given by Bryce
Routing:
- net 3.3V: track 73.9 -> 81.4 mm
- net N$10: track 9.46 -> 13.0 mm
- net 5.2V: track 93.3 -> 94.8 mm
Changed lines of the file:
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@@
 <wire x1="43.18" y1="3.81" x2="40.64" y2="3.81" width="0.6858" layer="1"/>
 <wire x1="5.588" y1="24.13" x2="15.24" y2="24.13" width="0.508" layer="16"/>
-<wire x1="18.37" y1="17.78" x2="18.37" y2="15.92" width="0.508" layer="1"/>
-<wire x1="18.37" y1="15.92" x2="22.86" y2="11.43" width="0.508" layer="1"/>
-<wire x1="22.86" y1="11.43" x2="22.86" y2="6.35" width="0.508" layer="1"/>
-<wire x1="22.86" y1="6.35" x2="24.13" y2="5.08" width="0.508" layer="1"/>
 <wire x1="15.24" y1="24.13" x2="18.37" y2="24.13" width="0.508" layer="1"/>
 <wire x1="24.13" y1="37.25" x2="22.44" y2="35.56" width="0.508" layer="1"/>
@@
 <wire x1="20.32" y1="35.56" x2="18.37" y2="33.61" width="0.508" layer="1"/>
 <wire x1="18.37" y1="33.61" x2="18.37" y2="30.48" width="0.508" layer="1"/>
+<wire x1="18.37" y1="17.78" x2="19.05" y2="17.1" width="0.6858" layer="1"/>
+<wire x1="19.05" y1="17.1" x2="19.05" y2="13.97" width="0.6858" layer="1"/>
+<wire x1="19.05" y1="13.97" x2="20.32" y2="12.7" width="0.6858" layer="1"/>
+<wire x1="20.32" y1="12.7" x2="22.86" y2="12.7" width="0.6858" layer="1"/>
+<wire x1="22.86" y1="12.7" x2="24.13" y2="11.43" width="0.6858" layer="1"/>
+<wire x1="24.13" y1="11.43" x2="24.13" y2="5.08" width="0.6858" layer="1"/>
 </signal>
 <signal name="12V">
@@
 <contactref element="U1" pad="2"/>
 <wire x1="7.62" y1="27.09" x2="7.62" y2="20.98" width="0.6858" layer="1"/>
-<wire x1="7.62" y1="20.98" x2="9.5" y2="22.86" width="0.6858" layer="1"/>
-<wire x1="12.7" y1="21.59" x2="12.7" y2="13.97" width="0.6858" layer="1"/>
-<via x="12.7" y="13.97" extent="1-16" drill="0.35"/>
-<via x="17.78" y="13.97" extent="1-16" drill="0.35"/>
-<wire x1="17.78" y1="13.97" x2="18.2" y2="13.55" width="0.6858" layer="1"/>
-<wire x1="18.2" y1="13.55" x2="18.2" y2="11.43" width="0.6858" layer="1"/>
-<wire x1="9.5" y1="22.86" x2="11.43" y2="22.86" width="0.6858" layer="1"/>
 <wire x1="7.62" y1="27.09" x2="5.93" y2="27.09" width="0.6858" layer="1"/>
 <wire x1="5.93" y1="27.09" x2="5.08" y2="27.94" width="0.6858" layer="1"/>
@@
 <wire x1="43.18" y1="6.35" x2="43.18" y2="8.89" width="0.6858" layer="1"/>
 <via x="43.18" y="8.89" extent="1-16" drill="0.35"/>
-<via x="17.78" y="8.89" extent="1-16" drill="0.35"/>
-<wire x1="12.7" y1="13.97" x2="17.78" y2="13.97" width="0.508" layer="16"/>
-<wire x1="18.2" y1="11.43" x2="17.78" y2="11.01" width="0.508" layer="1"/>
-<wire x1="17.78" y1="11.01" x2="17.78" y2="8.89" width="0.508" layer="1"/>
-<wire x1="17.78" y1="8.89" x2="43.18" y2="8.89" width="0.508" layer="16"/>
-<wire x1="11.43" y1="22.86" x2="12.7" y2="21.59" width="0.6858" layer="1"/>
+<wire x1="18.2" y1="11.43" x2="18.2" y2="9.74" width="0.6858" layer="1"/>
+<wire x1="18.2" y1="9.74" x2="19.05" y2="8.89" width="0.6858" layer="1"/>
+<via x="19.05" y="8.89" extent="1-16" drill="0.35"/>
+<wire x1="19.05" y1="8.89" x2="43.18" y2="8.89" width="0.6858" layer="16"/>
+<wire x1="18.2" y1="11.43" x2="3.81" y2="11.43" width="0.6858" layer="1"/>
+<wire x1="3.81" y1="11.43" x2="2.54" y2="12.7" width="0.6858" layer="1"/>
+<via x="2.54" y="12.7" extent="1-16" drill="0.35"/>
+<wire x1="2.54" y1="12.7" x2="2.54" y2="19.05" width="0.6858" layer="16"/>
+<wire x1="2.54" y1="19.05" x2="6.35" y2="22.86" width="0.6858" layer="16"/>
+<via x="6.35" y="22.86" extent="1-16" drill="0.35"/>
+<wire x1="6.35" y1="22.86" x2="7.62" y2="21.59" width="0.6858" layer="1"/>
+<wire x1="7.62" y1="21.59" x2="7.62" y2="20.98" width="0.6858" layer="1"/>
 </signal>
 <signal name="CRADJ">
@@
 <contactref element="R9" pad="1"/>
 <contactref element="D7" pad="A"/>
-<wire x1="12.307" y1="10.16" x2="16.51" y2="10.16" width="0.6858" layer="1"/>
+<via x="20.32" y="7.62" extent="1-16" drill="0.35"/>
+<wire x1="19.9" y1="11.43" x2="19.9" y2="9.27531875" width="0.6858" layer="1"/>
+<wire x1="19.9" y1="9.27531875" x2="19.9235" y2="9.25181875" width="0.6858" layer="1"/>
+<wire x1="19.9235" y1="8.0165" x2="20.32" y2="7.62" width="0.6858" layer="1"/>
+<wire x1="19.9235" y1="9.25181875" x2="19.9235" y2="8.0165" width="0.6858" layer="1"/>
+<wire x1="20.32" y1="7.62" x2="19.05" y2="7.62" width="0.6858" layer="16"/>
+<wire x1="19.05" y1="7.62" x2="16.51" y2="10.16" width="0.6858" layer="16"/>
 <via x="16.51" y="10.16" extent="1-16" drill="0.35"/>
-<via x="20.32" y="10.16" extent="1-16" drill="0.35"/>
-<wire x1="16.51" y1="10.16" x2="20.32" y2="10.16" width="0.508" layer="16"/>
-<wire x1="20.32" y1="10.16" x2="19.9" y2="10.58" width="0.508" layer="1"/>
-<wire x1="19.9" y1="10.58" x2="19.9" y2="11.43" width="0.508" layer="1"/>
+<wire x1="16.51" y1="10.16" x2="12.307" y2="10.16" width="0.6858" layer="1"/>
 </signal>
 <signal name="SWITCH">
@@
 <wire x1="26.67" y1="37.25" x2="26.67" y2="34.29" width="0.6858" layer="1"/>
 <wire x1="26.67" y1="34.29" x2="31.75" y2="29.21" width="0.6858" layer="1"/>
-<wire x1="31.75" y1="29.21" x2="33.02" y2="29.21" width="0.6858" layer="1"/>
-<wire x1="38.162" y1="32.358" x2="36.168" y2="32.358" width="0.254" layer="1"/>
-<wire x1="36.168" y1="32.358" x2="33.02" y2="29.21" width="0.6858" layer="1"/>
 <wire x1="24.13" y1="41.91" x2="26.67" y2="41.91" width="0.6858" layer="1"/>
 <wire x1="26.67" y1="41.91" x2="29.21" y2="39.37" width="0.6858" layer="1"/>
@@
 <wire x1="38.162" y1="32.358" x2="38.162" y2="27.128" width="0.6858" layer="1"/>
 <wire x1="38.162" y1="27.128" x2="40.64" y2="24.65" width="0.6858" layer="1"/>
+<wire x1="35.014" y1="29.21" x2="38.162" y2="32.358" width="0.6858" layer="1"/>
+<wire x1="31.75" y1="29.21" x2="35.014" y2="29.21" width="0.6858" layer="1"/>
 </signal>
 </signals>

Commit message: Edited some minor adj
Parts:
- moved DIODE 21.6 mm to (16.5, 34.3), turned to 180 degrees
- moved L1 18.2 mm to (22.9, 22.9)
- moved COUT1 16.5 mm to (38.1, 30.5)
- moved COUT2 16.5 mm to (38.1, 24.1)
- moved COUT3 16.5 mm to (38.1, 17.8)
- moved C11 12.3 mm to (7.24, 15.6), turned to 180 degrees
- moved R9 11.9 mm to (7.11, 11.4), turned to 0 degrees
- moved C10 11.6 mm to (11.0, 15.6)
- moved D7 8.23 mm to (3.30, 11.4)
- moved R7 4.02 mm to (48.3, 33.0), turned to 270 degrees
- moved U1 4.02 mm to (8.89, 21.6), turned to 0 degrees
- moved U$1 2.84 mm to (22.9, 44.5)
- moved CB 2.84 mm to (25.4, 40.6)
- moved CIN2 2.84 mm to (15.2, 40.6)
- moved R1 2.84 mm to (20.3, 40.6)
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Routing:
- net 12V: track 66.9 -> 9.77 mm
- net 5.2V: track 94.8 -> 40.5 mm
- net SWITCH: track 36.3 -> 21.1 mm
- net N$10: track 13.0 -> 2.08 mm, vias 2 -> 0
- net 3.3V: track 81.4 -> 72.0 mm, vias 4 -> 3
- net GND: track 12.7 -> 18.7 mm
- net N$8: track 7.39 -> 2.55 mm
- added copper zone on layer 16, net 12V
- added copper zone on layer 1, net 5.2V
- added copper zone on layer 1, net SWITCH

Commit message: Minh da best
Parts:
- moved D7 3.98 mm to (7.11, 10.3), turned to 0 degrees
- moved R9 1.27 mm to (7.11, 12.7)
Routing:
- net 5.2V: track 40.5 -> 35.7 mm
- net 3.3V: track 72.0 -> 71.3 mm
Changed lines of the file:
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@@
 <attribute name="VALUE" x="30.48" y="6.858" size="0.6096" layer="27" font="vector" ratio="20" align="top-center"/>
 </element>
-<element name="R9" library="SparkFun-Resistors" library_urn="urn:adsk.eagle:library:532" package="0603" package3d_urn="urn:adsk.eagle:package:39650/1" value="200" x="7.112" y="11.43" smashed="yes">
-<attribute name="NAME" x="7.112" y="12.192" size="0.6096" layer="25" font="vector" ratio="20" align="bottom-center"/>
-<attribute name="PROD_ID" value="RES-07862" x="-13.208" y="8.89" size="1.778" layer="27" display="off"/>
-<attribute name="VALUE" x="7.112" y="10.668" size="0.6096" layer="27" font="vector" ratio="20" align="top-center"/>
+<element name="R9" library="SparkFun-Resistors" library_urn="urn:adsk.eagle:library:532" package="0603" package3d_urn="urn:adsk.eagle:package:39650/1" value="200" x="7.112" y="12.7" smashed="yes">
+<attribute name="NAME" x="7.112" y="13.462" size="0.6096" layer="25" font="vector" ratio="20" align="bottom-center"/>
+<attribute name="PROD_ID" value="RES-07862" x="-13.208" y="10.16" size="1.778" layer="27" display="off"/>
+<attribute name="VALUE" x="7.112" y="11.938" size="0.6096" layer="27" font="vector" ratio="20" align="top-center"/>
 </element>
 <element name="D6" library="SparkFun-LED" library_urn="urn:adsk.eagle:library:529" package="LED-0603" package3d_urn="urn:adsk.eagle:package:39354/1" value="RED" x="29.591" y="4.572" smashed="yes" rot="R270">
@@
 <attribute name="VALUE" x="28.956" y="4.572" size="0.6096" layer="27" font="vector" ratio="20" rot="R270" align="top-center"/>
 </element>
-<element name="D7" library="SparkFun-LED" library_urn="urn:adsk.eagle:library:529" package="LED-0603" package3d_urn="urn:adsk.eagle:package:39354/1" value="BLUE" x="3.302" y="11.43" smashed="yes" rot="R180">
-<attribute name="NAME" x="3.302" y="10.795" size="0.6096" layer="25" font="vector" ratio="20" rot="R180" align="bottom-center"/>
-<attribute name="PROD_ID" value="DIO-08575" x="35.052" y="21.59" size="1.778" layer="27" rot="R180" display="off"/>
-<attribute name="VALUE" x="3.302" y="12.065" size="0.6096" layer="27" font="vector" ratio="20" rot="R180" align="top-center"/>
+<element name="D7" library="SparkFun-LED" library_urn="urn:adsk.eagle:library:529" package="LED-0603" package3d_urn="urn:adsk.eagle:package:39354/1" value="BLUE" x="7.112" y="10.287" smashed="yes">
+<attribute name="NAME" x="7.112" y="10.922" size="0.6096" layer="25" font="vector" ratio="20" align="bottom-center"/>
+<attribute name="PROD_ID" value="DIO-08575" x="-24.638" y="0.127" size="1.778" layer="27" display="off"/>
+<attribute name="VALUE" x="7.112" y="9.652" size="0.6096" layer="27" font="vector" ratio="20" align="top-center"/>
 </element>
 <element name="CIN1" library="X15-Conversion-Parts-Library" package="CAP_EEEFKE181XSP" value="180uF" x="7.62" y="44.45" smashed="yes" rot="R180">
@@
 <contactref element="COUT3" pad="+"/>
 <contactref element="L1" pad="2"/>
-<wire x1="15.24" y1="15.24" x2="16.51" y2="13.97" width="0.6858" layer="1"/>
-<wire x1="16.51" y1="13.97" x2="20.32" y2="13.97" width="0.6858" layer="1"/>
-<wire x1="20.32" y1="13.97" x2="22.86" y2="16.51" width="0.6858" layer="1"/>
-<wire x1="22.86" y1="16.51" x2="22.86" y2="17.26" width="0.6858" layer="1"/>
 <wire x1="34.88" y1="30.48" x2="34.88" y2="37.51" width="0.6858" layer="1"/>
 <wire x1="34.88" y1="37.51" x2="34.29" y2="38.1" width="0.6858" layer="1"/>
@@
 <wire x1="11.899" y1="15.621" x2="11.899" y2="17.681" width="0.6858" layer="1"/>
 <wire x1="11.899" y1="17.681" x2="11.19" y2="18.39" width="0.6858" layer="1"/>
-<wire x1="15.24" y1="17.12" x2="15.24" y2="15.24" width="0.6858" layer="1"/>
-<wire x1="11.19" y1="18.39" x2="13.97" y2="18.39" width="0.6858" layer="1"/>
-<wire x1="13.97" y1="18.39" x2="15.24" y2="17.12" width="0.6858" layer="1"/>
+<wire x1="11.899" y1="15.621" x2="21.221" y2="15.621" width="0.6858" layer="1"/>
+<wire x1="21.221" y1="15.621" x2="22.86" y2="17.26" width="0.6858" layer="1"/>
 </signal>
 <signal name="12V">
@@
 <contactref element="R9" pad="2"/>
 <contactref element="U1" pad="2"/>
-<wire x1="7.962" y1="11.43" x2="16.51" y2="11.43" width="0.6858" layer="1"/>
+<wire x1="15.24" y1="12.7" x2="16.51" y2="11.43" width="0.6858" layer="1"/>
+<wire x1="15.24" y1="12.7" x2="7.962" y2="12.7" width="0.6858" layer="1"/>
 <via x="16.51" y="11.43" extent="1-16" drill="0.35"/>
 <wire x1="16.51" y1="11.43" x2="44.45" y2="11.43" width="0.6858" layer="16"/>
@@
 <wire x1="45.72" y1="10.16" x2="45.72" y2="3.81" width="0.6858" layer="16"/>
 <wire x1="45.72" y1="3.81" x2="48.26" y2="3.81" width="0.6858" layer="16"/>
-<wire x1="7.962" y1="11.43" x2="7.962" y2="15.494" width="0.6858" layer="1"/>
+<wire x1="7.962" y1="12.7" x2="7.962" y2="15.494" width="0.6858" layer="1"/>
 <wire x1="7.962" y1="15.494" x2="8.089" y2="15.621" width="0.6858" layer="1"/>
 <wire x1="8.089" y1="15.621" x2="8.089" y2="17.589" width="0.6858" layer="1"/>
@@
 <contactref element="R9" pad="1"/>
 <contactref element="D7" pad="A"/>
-<wire x1="4.179" y1="11.43" x2="6.262" y2="11.43" width="0.6858" layer="1"/>
+<wire x1="6.262" y1="12.7" x2="6.262" y2="10.314" width="0.6858" layer="1"/>
+<wire x1="6.262" y1="10.314" x2="6.235" y2="10.287" width="0.6858" layer="1"/>
 </signal>
 <signal name="SWITCH">

Commit message: added test points
Parts:
- added J1, J2, J3: (no value), SparkFun-Connectors:1X02
Connections:
- net 3.3V: now also J2.1, J2.2
- net 5.2V: now also J3.1, J3.2
- net GND: now also J1.1, J1.2
Changed lines of the file:
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@@
 <attribute name="VALUE" x="15.24" y="21.59" size="1.27" layer="27" rot="R270" align="top-center"/>
+</element>
+<element name="J1" library="SparkFun-Connectors" library_urn="urn:adsk.eagle:library:513" package="1X02" package3d_urn="urn:adsk.eagle:package:38039/1" value="" x="48.895" y="18.288" smashed="yes" rot="R90">
+<attribute name="NAME" x="47.498" y="17.018" size="0.6096" layer="25" font="vector" ratio="20" rot="R90"/>
+<attribute name="VALUE" x="50.927" y="17.018" size="0.6096" layer="27" font="vector" ratio="20" rot="R90"/>
+</element>
+<element name="J2" library="SparkFun-Connectors" library_urn="urn:adsk.eagle:library:513" package="1X02" package3d_urn="urn:adsk.eagle:package:38039/1" value="" x="3.175" y="24.638" smashed="yes" rot="R90">
+<attribute name="NAME" x="1.778" y="23.368" size="0.6096" layer="25" font="vector" ratio="20" rot="R90"/>
+<attribute name="VALUE" x="5.207" y="23.368" size="0.6096" layer="27" font="vector" ratio="20" rot="R90"/>
+</element>
+<element name="J3" library="SparkFun-Connectors" library_urn="urn:adsk.eagle:library:513" package="1X02" package3d_urn="urn:adsk.eagle:package:38039/1" value="" x="3.175" y="11.938" smashed="yes" rot="R90">
+<attribute name="NAME" x="1.778" y="10.668" size="0.6096" layer="25" font="vector" ratio="20" rot="R90"/>
+<attribute name="VALUE" x="5.207" y="10.668" size="0.6096" layer="27" font="vector" ratio="20" rot="R90"/>
 </element>
 </elements>
@@
 <vertex x="-3.81" y="67.31"/>
 <vertex x="58.42" y="67.31"/>
-<vertex x="60.96" y="64.77"/>
 <vertex x="66.04" y="59.69"/>
 <vertex x="66.04" y="8.89"/>
 <vertex x="49.53" y="-7.62"/>
 <vertex x="11.43" y="-7.62"/>
-<vertex x="-11.43" y="-7.62"/>
-<vertex x="-13.97" y="-5.08"/>
+<vertex x="33.811734375" y="14.761734375"/>
+<vertex x="28.418265625" y="14.761734375"/>
 <vertex x="-13.97" y="57.15"/>
-<vertex x="-8.89" y="62.23"/>
 </polygon>
 <contactref element="DIODE" pad="2"/>
@@
 <wire x1="29.591" y1="3.695" x2="29.706" y2="3.81" width="0.6858" layer="1"/>
 <wire x1="29.706" y1="3.81" x2="35.56" y2="3.81" width="0.6858" layer="1"/>
+<contactref element="J1" pad="2"/>
+<contactref element="J1" pad="1"/>
+<wire x1="19.05" y1="52.105" x2="30.48" y2="58.42" width="0" layer="19" extent="1-1"/>
+<wire x1="19.05" y1="44.45" x2="19.05" y2="52.105" width="0" layer="19" extent="1-1"/>
+<wire x1="20.32" y1="39.79" x2="19.05" y2="44.45" width="0" layer="19" extent="1-1"/>
+<wire x1="17.78" y1="39.79" x2="20.32" y2="39.79" width="0" layer="19" extent="1-1"/>
+<wire x1="15.24" y1="39.79" x2="17.78" y2="39.79" width="0" layer="19" extent="1-1"/>
+<wire x1="12.812" y1="34.352" x2="15.24" y2="39.79" width="0" layer="19" extent="1-1"/>
+<wire x1="8.89" y1="24.79" x2="12.812" y2="34.352" width="0" layer="19" extent="1-1"/>
+<wire x1="6.59" y1="18.39" x2="8.89" y2="24.79" width="0" layer="19" extent="1-1"/>
+<wire x1="6.389" y1="15.621" x2="6.59" y2="18.39" width="0" layer="19" extent="1-1"/>
+<wire x1="10.199" y1="15.621" x2="6.389" y2="15.621" width="0" layer="19" extent="1-1"/>
+<wire x1="7.989" y1="10.287" x2="6.389" y2="15.621" width="0" layer="19" extent="1-1"/>
+<wire x1="5.08" y1="5.08" x2="7.989" y2="10.287" width="0" layer="19" extent="1-1"/>
+<wire x1="15.24" y1="5.08" x2="7.989" y2="10.287" width="0" layer="19" extent="1-1"/>
+<wire x1="5.12" y1="44.45" x2="15.24" y2="39.79" width="0" layer="19" extent="1-1"/>
+<wire x1="29.591" y1="3.695" x2="15.24" y2="5.08" width="0" layer="19" extent="1-1"/>
+<wire x1="38.1" y1="3.81" x2="35.56" y2="3.81" width="0" layer="19" extent="1-1"/>
+<wire x1="41.32" y1="17.78" x2="38.1" y2="3.81" width="0" layer="19" extent="1-1"/>
+<wire x1="45.72" y1="32.143" x2="41.32" y2="30.48" width="0" layer="19" extent="1-1"/>
+<wire x1="40.64" y1="44.45" x2="45.72" y2="32.143" width="0" layer="19" extent="1-1"/>
+<wire x1="38.1" y1="44.45" x2="40.64" y2="44.45" width="0" layer="19" extent="1-1"/>
+<wire x1="48.895" y1="20.828" x2="5.08" y2="5.08" width="0" layer="19" extent="1-1"/>
+<wire x1="48.895" y1="18.288" x2="48.895" y2="20.828" width="0" layer="19" extent="1-1"/>
 </signal>
 <signal name="5.2V">
@@
 <wire x1="11.899" y1="15.621" x2="21.221" y2="15.621" width="0.6858" layer="1"/>
 <wire x1="21.221" y1="15.621" x2="22.86" y2="17.26" width="0.6858" layer="1"/>
+<contactref element="J3" pad="2"/>
+<contactref element="J3" pad="1"/>
+<wire x1="34.88" y1="24.13" x2="34.88" y2="30.48" width="0" layer="19" extent="1-1"/>
+<wire x1="34.88" y1="17.78" x2="34.88" y2="24.13" width="0" layer="19" extent="1-1"/>
+<wire x1="31.33" y1="7.62" x2="34.88" y2="17.78" width="0" layer="19" extent="1-1"/>
+<wire x1="24.13" y1="5.08" x2="31.33" y2="7.62" width="0" layer="19" extent="1-1"/>
+<wire x1="40.64" y1="3.81" x2="31.33" y2="7.62" width="0" layer="19" extent="1-1"/>
+<wire x1="43.18" y1="3.81" x2="40.64" y2="3.81" width="0" layer="19" extent="1-1"/>
+<wire x1="22.86" y1="17.26" x2="34.88" y2="17.78" width="0" layer="19" extent="1-1"/>
+<wire x1="3.175" y1="14.478" x2="11.899" y2="15.621" width="0" layer="19" extent="1-1"/>
+<wire x1="3.175" y1="11.938" x2="3.175" y2="14.478" width="0" layer="19" extent="1-1"/>
 </signal>
 <signal name="12V">
@@
 <vertex x="13.97" y="59.69"/>
 </polygon>
-<via x="13.97" y="44.45" extent="1-16" drill="0.35"/>
+<via x="13.97" y="44.45" extent="1-16" drill="0.55"/>
 <wire x1="48.26" y1="32.17" x2="48.26" y2="30.48" width="0.6858" layer="1"/>
 <via x="48.26" y="30.48" extent="1-16" drill="0.35"/>
+<wire x1="43.18" y1="44.45" x2="45.72" y2="44.45" width="0" layer="19" extent="1-1"/>
+<wire x1="46.99" y1="39.37" x2="45.72" y2="44.45" width="0" layer="19" extent="1-1"/>
+<wire x1="48.26" y1="32.17" x2="46.99" y2="39.37" width="0" layer="19" extent="1-1"/>
+<wire x1="15.24" y1="44.45" x2="43.18" y2="44.45" width="0" layer="19" extent="1-1"/>
 </signal>
 <signal name="3.3V">
@@
 <via x="8.89" y="21.59" extent="1-16" drill="0.35"/>
 <wire x1="8.89" y1="21.59" x2="8.89" y2="18.39" width="0.6858" layer="1"/>
+<contactref element="J2" pad="2"/>
+<contactref element="J2" pad="1"/>
+<wire x1="3.175" y1="27.178" x2="3.175" y2="24.638" width="0" layer="19" extent="1-1"/>
+<wire x1="7.962" y1="12.7" x2="3.175" y2="27.178" width="0" layer="19" extent="1-1"/>
 </signal>
 <signal name="CRADJ">
