File: X15-Conversion.brd (EAGLE design)
At the start: 50.8 x 62.9 mm, 31 parts, among them U1 LINEAR,AZ1117CR-3.3TRG1DIODES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

Commit message: Chenaged some cool stuff you know
Parts:
- moved J2 0.77 mm to (3.05, 25.4)
- moved J3 0.57 mm to (2.92, 11.4)
Routing:
- net 5.2V: track 35.7 -> 48.6 mm, vias 2 -> 4
- net 3.3V: track 71.3 -> 79.6 mm
- net 12V: track 9.77 -> 1.69 mm
- added copper zone on layer 1, net 12V
Changed lines of the file:
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@@
 <attribute name="VALUE" x="50.927" y="17.018" size="0.6096" layer="27" font="vector" ratio="20" rot="R90"/>
 </element>
-<element name="J2" library="SparkFun-Connectors" library_urn="urn:adsk.eagle:library:513" package="1X02" package3d_urn="urn:adsk.eagle:package:38039/1" value="" x="3.175" y="24.638" smashed="yes" rot="R90">
-<attribute name="NAME" x="1.778" y="23.368" size="0.6096" layer="25" font="vector" ratio="20" rot="R90"/>
-<attribute name="VALUE" x="5.207" y="23.368" size="0.6096" layer="27" font="vector" ratio="20" rot="R90"/>
+<element name="J2" library="SparkFun-Connectors" library_urn="urn:adsk.eagle:library:513" package="1X02" package3d_urn="urn:adsk.eagle:package:38039/1" value="" x="3.048" y="25.4" smashed="yes" rot="R90">
+<attribute name="NAME" x="1.651" y="24.13" size="0.6096" layer="25" font="vector" ratio="20" rot="R90"/>
+<attribute name="VALUE" x="5.08" y="24.13" size="0.6096" layer="27" font="vector" ratio="20" rot="R90"/>
 </element>
-<element name="J3" library="SparkFun-Connectors" library_urn="urn:adsk.eagle:library:513" package="1X02" package3d_urn="urn:adsk.eagle:package:38039/1" value="" x="3.175" y="11.938" smashed="yes" rot="R90">
-<attribute name="NAME" x="1.778" y="10.668" size="0.6096" layer="25" font="vector" ratio="20" rot="R90"/>
-<attribute name="VALUE" x="5.207" y="10.668" size="0.6096" layer="27" font="vector" ratio="20" rot="R90"/>
+<element name="J3" library="SparkFun-Connectors" library_urn="urn:adsk.eagle:library:513" package="1X02" package3d_urn="urn:adsk.eagle:package:38039/1" value="" x="2.921" y="11.43" smashed="yes" rot="R90">
+<attribute name="NAME" x="1.524" y="10.16" size="0.6096" layer="25" font="vector" ratio="20" rot="R90"/>
+<attribute name="VALUE" x="4.953" y="10.16" size="0.6096" layer="27" font="vector" ratio="20" rot="R90"/>
 </element>
 </elements>
@@
 <contactref element="U1" pad="4"/>
 <contactref element="U1" pad="1"/>
-<polygon width="0.1524" layer="1" rank="6">
+<polygon width="0.1524" layer="1" isolate="0.2032" rank="6">
 <vertex x="38.1" y="64.77"/>
 <vertex x="38.1" y="60.96"/>
@@
 <vertex x="-3.81" y="62.23"/>
 <vertex x="-1.27" y="64.77"/>
-</polygon>
-<polygon width="0.1524" layer="16" rank="6">
-<vertex x="-3.81" y="67.31"/>
-<vertex x="58.42" y="67.31"/>
-<vertex x="66.04" y="59.69"/>
-<vertex x="66.04" y="8.89"/>
-<vertex x="49.53" y="-7.62"/>
-<vertex x="11.43" y="-7.62"/>
-<vertex x="33.811734375" y="14.761734375"/>
-<vertex x="28.418265625" y="14.761734375"/>
-<vertex x="-13.97" y="57.15"/>
 </polygon>
 <contactref element="DIODE" pad="2"/>
@@
 <contactref element="J1" pad="2"/>
 <contactref element="J1" pad="1"/>
-<wire x1="19.05" y1="52.105" x2="30.48" y2="58.42" width="0" layer="19" extent="1-1"/>
-<wire x1="19.05" y1="44.45" x2="19.05" y2="52.105" width="0" layer="19" extent="1-1"/>
-<wire x1="20.32" y1="39.79" x2="19.05" y2="44.45" width="0" layer="19" extent="1-1"/>
-<wire x1="17.78" y1="39.79" x2="20.32" y2="39.79" width="0" layer="19" extent="1-1"/>
-<wire x1="15.24" y1="39.79" x2="17.78" y2="39.79" width="0" layer="19" extent="1-1"/>
-<wire x1="12.812" y1="34.352" x2="15.24" y2="39.79" width="0" layer="19" extent="1-1"/>
-<wire x1="8.89" y1="24.79" x2="12.812" y2="34.352" width="0" layer="19" extent="1-1"/>
-<wire x1="6.59" y1="18.39" x2="8.89" y2="24.79" width="0" layer="19" extent="1-1"/>
-<wire x1="6.389" y1="15.621" x2="6.59" y2="18.39" width="0" layer="19" extent="1-1"/>
-<wire x1="10.199" y1="15.621" x2="6.389" y2="15.621" width="0" layer="19" extent="1-1"/>
-<wire x1="7.989" y1="10.287" x2="6.389" y2="15.621" width="0" layer="19" extent="1-1"/>
-<wire x1="5.08" y1="5.08" x2="7.989" y2="10.287" width="0" layer="19" extent="1-1"/>
-<wire x1="15.24" y1="5.08" x2="7.989" y2="10.287" width="0" layer="19" extent="1-1"/>
-<wire x1="5.12" y1="44.45" x2="15.24" y2="39.79" width="0" layer="19" extent="1-1"/>
-<wire x1="29.591" y1="3.695" x2="15.24" y2="5.08" width="0" layer="19" extent="1-1"/>
-<wire x1="38.1" y1="3.81" x2="35.56" y2="3.81" width="0" layer="19" extent="1-1"/>
-<wire x1="41.32" y1="17.78" x2="38.1" y2="3.81" width="0" layer="19" extent="1-1"/>
-<wire x1="45.72" y1="32.143" x2="41.32" y2="30.48" width="0" layer="19" extent="1-1"/>
-<wire x1="40.64" y1="44.45" x2="45.72" y2="32.143" width="0" layer="19" extent="1-1"/>
-<wire x1="38.1" y1="44.45" x2="40.64" y2="44.45" width="0" layer="19" extent="1-1"/>
-<wire x1="48.895" y1="20.828" x2="5.08" y2="5.08" width="0" layer="19" extent="1-1"/>
-<wire x1="48.895" y1="18.288" x2="48.895" y2="20.828" width="0" layer="19" extent="1-1"/>
+<polygon width="0.1524" layer="16" isolate="0.2032" rank="6">
+<vertex x="-5.08" y="68.58"/>
+<vertex x="45.72" y="68.58"/>
+<vertex x="55.88" y="58.42"/>
+<vertex x="62.23" y="52.07"/>
+<vertex x="62.23" y="-3.81"/>
+<vertex x="55.88" y="-10.16"/>
+<vertex x="43.18" y="-10.16"/>
+<vertex x="-1.27" y="-10.16"/>
+<vertex x="-10.16" y="-1.27"/>
+<vertex x="-10.16" y="63.5"/>
+</polygon>
 </signal>
 <signal name="5.2V">
@@
 <contactref element="J3" pad="2"/>
 <contactref element="J3" pad="1"/>
-<wire x1="34.88" y1="24.13" x2="34.88" y2="30.48" width="0" layer="19" extent="1-1"/>
-<wire x1="34.88" y1="17.78" x2="34.88" y2="24.13" width="0" layer="19" extent="1-1"/>
-<wire x1="31.33" y1="7.62" x2="34.88" y2="17.78" width="0" layer="19" extent="1-1"/>
-<wire x1="24.13" y1="5.08" x2="31.33" y2="7.62" width="0" layer="19" extent="1-1"/>
-<wire x1="40.64" y1="3.81" x2="31.33" y2="7.62" width="0" layer="19" extent="1-1"/>
-<wire x1="43.18" y1="3.81" x2="40.64" y2="3.81" width="0" layer="19" extent="1-1"/>
-<wire x1="22.86" y1="17.26" x2="34.88" y2="17.78" width="0" layer="19" extent="1-1"/>
-<wire x1="3.175" y1="14.478" x2="11.899" y2="15.621" width="0" layer="19" extent="1-1"/>
-<wire x1="3.175" y1="11.938" x2="3.175" y2="14.478" width="0" layer="19" extent="1-1"/>
+<wire x1="2.921" y1="11.43" x2="2.921" y2="13.97" width="0.6858" layer="1"/>
+<wire x1="5.08" y1="13.97" x2="2.921" y2="13.97" width="0.6858" layer="1"/>
+<via x="5.08" y="13.97" extent="1-16" drill="0.35"/>
+<wire x1="5.08" y1="13.97" x2="11.43" y2="13.97" width="0.6858" layer="16"/>
+<via x="11.43" y="13.97" extent="1-16" drill="0.35"/>
+<wire x1="11.43" y1="13.97" x2="11.899" y2="14.439" width="0.6858" layer="1"/>
+<wire x1="11.899" y1="14.439" x2="11.899" y2="15.621" width="0.6858" layer="1"/>
 </signal>
 <signal name="12V">
@@
 <contactref element="R7" pad="2"/>
 <contactref element="CIN1" pad="1"/>
-<wire x1="15.24" y1="44.45" x2="13.97" y2="44.45" width="0.6858" layer="1"/>
-<wire x1="13.97" y1="44.45" x2="10.12" y2="44.45" width="0.6858" layer="1"/>
-<wire x1="15.24" y1="41.49" x2="15.24" y2="44.45" width="0.508" layer="1"/>
 <polygon width="0.2032" layer="16">
-<vertex x="12.7" y="58.42"/>
+<vertex x="12.7" y="62.23"/>
 <vertex x="12.7" y="44.45"/>
 <vertex x="13.97" y="43.18"/>
@@
 <vertex x="50.8" y="45.72"/>
 <vertex x="49.53" y="46.99"/>
-<vertex x="26.67" y="46.99"/>
-<vertex x="25.4" y="48.26"/>
-<vertex x="25.4" y="58.42"/>
-<vertex x="24.13" y="59.69"/>
-<vertex x="13.97" y="59.69"/>
+<vertex x="35.814" y="46.99"/>
+<vertex x="35.56" y="47.244"/>
+<vertex x="35.56" y="62.23"/>
 </polygon>
 <via x="13.97" y="44.45" extent="1-16" drill="0.55"/>
 <wire x1="48.26" y1="32.17" x2="48.26" y2="30.48" width="0.6858" layer="1"/>
 <via x="48.26" y="30.48" extent="1-16" drill="0.35"/>
-<wire x1="43.18" y1="44.45" x2="45.72" y2="44.45" width="0" layer="19" extent="1-1"/>
-<wire x1="46.99" y1="39.37" x2="45.72" y2="44.45" width="0" layer="19" extent="1-1"/>
-<wire x1="48.26" y1="32.17" x2="46.99" y2="39.37" width="0" layer="19" extent="1-1"/>
-<wire x1="15.24" y1="44.45" x2="43.18" y2="44.45" width="0" layer="19" extent="1-1"/>
+<polygon width="0.1524" layer="1">
+<vertex x="15.621" y="45.847"/>
+<vertex x="15.621" y="41.021"/>
+<vertex x="13.843" y="41.021"/>
+<vertex x="13.843" y="42.926"/>
+<vertex x="13.462" y="43.307"/>
+<vertex x="8.128" y="43.307"/>
+<vertex x="8.001" y="43.434"/>
+<vertex x="8.001" y="45.847"/>
+</polygon>
 </signal>
 <signal name="3.3V">
@@
 <contactref element="J2" pad="2"/>
 <contactref element="J2" pad="1"/>
-<wire x1="3.175" y1="27.178" x2="3.175" y2="24.638" width="0" layer="19" extent="1-1"/>
-<wire x1="7.962" y1="12.7" x2="3.175" y2="27.178" width="0" layer="19" extent="1-1"/>
+<wire x1="3.048" y1="25.4" x2="3.048" y2="27.94" width="0.6858" layer="1"/>
+<wire x1="3.048" y1="27.94" x2="8.89" y2="27.94" width="0.6858" layer="1"/>
 </signal>
 <signal name="CRADJ">
